File: traffic-light/traffic-light.kicad_pcb (KiCad board)
At the start: 2 copper layers, 99.1 x 99.1 mm, 23 parts, among them J1 BATTERY, J10 Traffic_Light_4, J11 ICSP, J2 RFID-RC522_1, J3 RFID-RC522_2, J4 RFID-RC522_3, J5 RFID-RC522_4, J6 Ground, J7 Traffic_Light_1, J8 Traffic_Light_2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

Commit message: Added diode and switch.
Parts:
- added D2: 1N4007, Diode_THT:D_DO-41_SOD81_P10.16mm_Horizontal, F.Cu at (175.4, 96.3)
- added SW1: PWR, Connector_PinSocket_2.54mm:PinSocket_1x03_P2.54mm_Vertical, F.Cu at (166.2, 102.5)
- J10: value Traffic_Light_4 -> Traffic_LEDS-4; footprint Connector_PinHeader_2.54mm:PinHeader_1x03_P2.54mm_Vertical -> Connector_PinHeader_2.54mm:PinHeader_1x04_P2.54mm_Vertical
- J6: footprint Connector_PinHeader_2.54mm:PinHeader_1x04_P2.54mm_Horizontal -> Connector_PinHeader_2.54mm:PinHeader_1x04_P2.54mm_Vertical
- J7: value Traffic_Light_1 -> Traffic_LEDS-1; footprint Connector_PinHeader_2.54mm:PinHeader_1x03_P2.54mm_Vertical -> Connector_PinHeader_2.54mm:PinHeader_1x04_P2.54mm_Vertical
- J8: value Traffic_Light_2 -> Traffic_LEDS-2; footprint Connector_PinHeader_2.54mm:PinHeader_1x03_P2.54mm_Vertical -> Connector_PinHeader_2.54mm:PinHeader_1x04_P2.54mm_Vertical
- J9: value Traffic_Light_3 -> Traffic_LEDS-3; footprint Connector_PinHeader_2.54mm:PinHeader_1x03_P2.54mm_Vertical -> Connector_PinHeader_2.54mm:PinHeader_1x04_P2.54mm_Vertical
- moved C1 13.2 mm to (189.1, 103.2), turned to 270 degrees
Connections:
- C1 pad 1: +BATT -> Net-(C1-Pad1)
- U1 pad 3: +BATT -> Net-(C1-Pad1)
Routing:
- net /cardDetected: track 143.0 -> 93.8 mm, vias 0 -> 2
- net Net-(C1-Pad1): track 0.00 -> 27.0 mm
- net Net-(D2-Pad1): track 0.00 -> 23.2 mm
- net +3V3: track 52.6 -> 39.6 mm
- net GND: track 37.7 -> 44.6 mm
- net +BATT: track 105.7 -> 110.1 mm
- net SS3: track 46.9 -> 45.7 mm
- net /cardSelect1: track 66.5 -> 65.6 mm
- net SS4: track 33.4 -> 32.7 mm
- net SS2: track 58.6 -> 58.0 mm
Other:
- net class Default: clearance 0.2 -> 0.4; trace_width 0.25 -> 0.8
- rule trace_clearance: 0.2 -> 0.4

Commit message: PCB corrections.
Parts:
- moved A1 9.20 mm to (109.7, 121.2)
- moved D1 7.27 mm to (121.4, 97.5)
- moved R1 4.48 mm to (134.1, 93.3)
- moved SW1 3.96 mm to (169.4, 100.2), turned to 180 degrees
- moved J2 3.83 mm to (192.5, 140.3)
- moved J3 3.83 mm to (184.9, 140.3)
- moved J4 3.83 mm to (177.3, 140.3)
- moved J5 3.83 mm to (169.7, 140.3)
- moved C6 3.02 mm to (149.8, 93.5)
- moved C2 0.43 mm to (185.0, 111.8), turned to 0 degrees
Connections:
- D2 pad 1: Net-(D2-Pad1) -> +BATT
- D2 pad 2: +BATT -> Net-(D2-Pad2)
- J1 pad 1: +BATT -> Net-(D2-Pad2)
- SW1 pad 2: Net-(D2-Pad1) -> +BATT
Routing:
- net GND: track 44.6 -> 108.7 mm, vias 2 -> 0
- net Net-(D2-Pad1): track 23.2 -> 0.00 mm
- net +BATT: track 110.1 -> 89.0 mm, vias 0 -> 2
- net SS1: track 70.3 -> 87.1 mm
- net SS2: track 58.0 -> 72.4 mm
- net /cardSelect1: track 65.6 -> 80.1 mm, vias 0 -> 2
- net /cardSelect0: track 64.9 -> 77.5 mm, vias 0 -> 2
- net SS3: track 45.7 -> 58.1 mm
- net SS4: track 32.7 -> 44.0 mm
- net Net-(D2-Pad2): track 0.00 -> 11.0 mm
- net /SCK: track 55.4 -> 66.3 mm
- net /MISO: track 41.4 -> 52.0 mm
- net /MOSI: track 46.9 -> 55.6 mm
- net /LED: track 60.8 -> 68.7 mm, vias 2 -> 0
- net /cardDetected: track 93.8 -> 88.7 mm
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Other:
- board text added: "Bahtiyar Bayram İbrahim Ethem Dere BTÜ -Traffic Light Controller"
- board text removed: "Bahtiyar Bayram İbrahim Ethem Dere BTÜ - Traffic Light Control"
